File: PCB/hackpad.kicad_pcb (KiCad board)
At the start: 2 copper layers, 61.9 x 59.5 mm, 8 parts, among them SW1 SW_Push, SW2 SW_Push, SW3 SW_Push, SW4 SW_Push, SW5 SW_Push, U1 XIAO-RP2040-DIP

Commit message: Add files via upload
Parts:
- removed D1, D2: SK6812MINI, LED_SMD:LED_SK6812MINI_PLCC4_3.5x3.5mm_P1.75mm
- added D3: SK6812MINI-E, SK6812MINIE:SK6812MINI-E_fixed, B.Cu at (164.3, 76.2)
- added D4: SK6812MINI-E, SK6812MINIE:SK6812MINI-E_fixed, B.Cu at (176.2, 61.9)
Routing:
- net Net-(D1-VSS): track 34.3 -> 0.00 mm
- net Net-(D3-DIN): track 0.00 -> 21.2 mm
- net Net-(D1-DOUT): track 17.8 -> 0.00 mm
- net Net-(D3-VSS): track 0.00 -> 15.8 mm
- net +5V: track 26.1 -> 39.5 mm
- net Net-(D4-DIN): track 34.6 -> 23.5 mm
